Commit message: bug fixes for real2sim and sim2real

File: wx250s.urdf (robot description, URDF)
Before this commit: robot wx250s, 14 links, 13 joints
Links:
- link gripper_prop_link: geometry visual mesh filename=meshes_wx250s/WXSA-250-M-8-Gripper-Prop.obj scale=0.001 0.001 0.001
Joints:
- joint right_finger: mimic joint=left_finger multiplier=1 offset=0 -> (none)
